File: hardware/ps2zx.kicad_pcb (KiCad board)
At the start: 2 copper layers, 55.9 x 38.1 mm, 12 parts, among them J1 Keyboard, J2 KB1, J3 KB2, J4 Board, J5 ISP, SW1 BTN1, SW2 BTN2, U1 ATmega8-16AU, Y1 16Mhz

Commit message: Revised version (not yet produced)
Parts:
- added D1: STATUS, LED_SMD:LED_0805_2012Metric_Pad1.15x1.40mm_HandSolder, F.Cu at (176.8, 120.4)
- added D2: POWER, LED_SMD:LED_0805_2012Metric_Pad1.15x1.40mm_HandSolder, F.Cu at (183.4, 120.4)
- added R1: 330Ω, Resistor_SMD:R_0805_2012Metric_Pad1.15x1.40mm_HandSolder, F.Cu at (176.3, 114.8)
- moved C1 13.4 mm to (164.6, 95.0), turned to 0 degrees
- turned U1 to 90 degrees
Connections:
- U1 pad 1: Net-(J3-Pad4) -> /~RDFE
- U1 pad 10: Net-(J3-Pad7) -> Net-(SW1-Pad1)
- U1 pad 11: Net-(J3-Pad8) -> Net-(SW2-Pad1)
- U1 pad 2: Net-(J3-Pad5) -> /~RESET
- U1 pad 23: /~RESET -> Net-(J3-Pad1)
- U1 pad 24: Net-(SW1-Pad1) -> Net-(J3-Pad2)
- U1 pad 25: Net-(SW2-Pad1) -> Net-(J3-Pad3)
- U1 pad 26: Net-(J3-Pad3) -> Net-(J3-Pad4)
- U1 pad 27: Net-(J1-Pad1) -> Net-(J3-Pad5)
- U1 pad 28: Net-(J1-Pad5) -> Net-(J3-Pad6)
- U1 pad 30: Net-(J3-Pad1) -> Net-(J3-Pad7)
- U1 pad 31: Net-(J3-Pad2) -> Net-(J3-Pad8)
- U1 pad 32: /~RDFE -> Net-(J1-Pad5)
- U1 pad 7: Net-(C3-Pad1) -> Net-(C2-Pad1)
- U1 pad 8: Net-(C2-Pad1) -> Net-(C3-Pad1)
- U1 pad 9: Net-(J3-Pad6) -> Net-(J1-Pad1)
- Y1 pad 1: Net-(C2-Pad1) -> Net-(C3-Pad1)
- Y1 pad 2: Net-(C3-Pad1) -> Net-(C2-Pad1)
Routing:
- net GND: track 138.8 -> 18.8 mm, vias 8 -> 4
- net /~RDFE: track 54.1 -> 22.0 mm, vias 3 -> 0
- net Net-(D1-Pad1): track 7.65 -> 34.9 mm, vias 0 -> 4
- net Net-(J2-Pad4): track 48.0 -> 21.1 mm, vias 4 -> 2
- net /~RESET: track 40.8 -> 23.4 mm, vias 3 -> 0
- net +5V: track 82.5 -> 97.2 mm, vias 3 -> 4
- net Net-(J3-Pad2): track 32.6 -> 18.0 mm, vias 4 -> 1
- net Net-(J2-Pad5): track 48.6 -> 34.1 mm, vias 3 -> 2
- net Net-(J3-Pad3): track 30.4 -> 16.6 mm, vias 2 -> 1
- net Net-(J3-Pad1): track 33.0 -> 22.4 mm
- net Net-(J2-Pad3): track 30.2 -> 20.6 mm, vias 1 -> 2
- net Net-(J2-Pad2): track 30.2 -> 21.4 mm
- net Net-(J3-Pad6): track 10.3 -> 17.4 mm, vias 1 -> 2
- net Net-(J2-Pad1): track 23.9 -> 17.9 mm, vias 1 -> 2
- net Net-(D1-Pad2): track 0.00 -> 5.80 mm
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- added copper zone on F.Cu, net GND
- removed copper zone on B.Cu, net GND

Commit message: Version 4 pre-production
Parts:
- added R2: 330Ω, Resistor_SMD:R_0805_2012Metric_Pad1.15x1.40mm_HandSolder, F.Cu at (184.4, 116.6)
- added REF**: MountingHole_2.2mm_M2, MountingHole:MountingHole_2.2mm_M2, F.Cu at (190.1, 121.5)
- added REF**: MountingHole_2.2mm_M2, MountingHole:MountingHole_2.2mm_M2, F.Cu at (140.1, 121.5)
- added REF**: MountingHole_2.2mm_M2, MountingHole:MountingHole_2.2mm_M2, F.Cu at (140.1, 89.3)
- added REF**: MountingHole_2.2mm_M2, MountingHole:MountingHole_2.2mm_M2, F.Cu at (190.1, 89.3)
- moved J3 35.6 mm to (182.9, 88.9), turned to 270 degrees
- moved J5 30.3 mm to (149.5, 114.6), turned to 90 degrees
- moved D1 15.4 mm to (189.5, 111.8), turned to 180 degrees
- moved J2 15.2 mm to (157.5, 88.9), turned to 270 degrees
- moved C2 10.8 mm to (150.1, 96.3)
- moved R1 8.68 mm to (184.4, 111.8)
- moved J1 7.37 mm to (173.2, 116.8)
- moved D2 7.19 mm to (189.5, 116.6), turned to 180 degrees
- moved U1 7.14 mm to (170.9, 102.4), turned to 270 degrees
- moved C1 6.29 mm to (170.8, 95.9), turned to 180 degrees
- moved Y1 6.27 mm to (155.2, 102.4)
- moved SW1 5.83 mm to (187.5, 105.4)
- moved SW2 4.56 mm to (187.5, 96.5)
- moved J4 2.54 mm to (139.7, 106.7)
- moved C3 2.41 mm to (150.1, 103.9)
Connections:
- D2 pad 2: +5V -> Net-(D2-Pad2)
Routing:
- net /~RDFE: track 22.0 -> 45.6 mm, vias 0 -> 2
- net Net-(J2-Pad4): track 21.1 -> 42.4 mm, vias 2 -> 1
- net /~RESET: track 23.4 -> 44.3 mm, vias 0 -> 2
- net +5V: track 97.2 -> 79.1 mm, vias 4 -> 5
- net Net-(J2-Pad5): track 34.1 -> 50.7 mm, vias 2 -> 3
- net Net-(SW1-Pad1): track 26.1 -> 41.4 mm, vias 0 -> 4
- net Net-(D1-Pad1): track 34.9 -> 49.5 mm, vias 4 -> 2
- net GND: track 18.8 -> 5.23 mm, vias 4 -> 0
- net Net-(J2-Pad3): track 20.6 -> 29.5 mm, vias 2 -> 1
- net Net-(J3-Pad1): track 22.4 -> 29.4 mm, vias 2 -> 1
- net Net-(J3-Pad2): track 18.0 -> 24.4 mm
- net Net-(C2-Pad1): track 27.7 -> 21.3 mm, vias 2 -> 0
- net Net-(J1-Pad1): track 17.9 -> 23.4 mm, vias 2 -> 1
- net Net-(SW2-Pad1): track 25.7 -> 30.7 mm, vias 0 -> 2
- net Net-(J3-Pad7): track 16.3 -> 21.2 mm
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Other:
- board text added: "PS/2 Keyboard to Jupiter Ace/ZX Spectrum Converter Version 4 github.com/hanshuebner/ps2zx"
- board text removed: "Version 3 github.com/hanshuebner/ps2zx"
