File: hardware/ps2zx.sch (KiCad schematic (older format))
At the start: 12 parts, among them J1 Keyboard, J2 KB1, J3 KB2, J4 Board, J5 ISP, SW1 BTN1, SW2 BTN2, U1 ATmega8-16AU, Y1 16Mhz

Commit message: Revised version (not yet produced)
Parts:
- added D1: STATUS, LED_SMD:LED_0805_2012Metric_Pad1.15x1.40mm_HandSolder, symbol Device:LED
- added D2: POWER, LED_SMD:LED_0805_2012Metric_Pad1.15x1.40mm_HandSolder, symbol Device:LED
- added R1: 330Ω, Resistor_SMD:R_0805_2012Metric_Pad1.15x1.40mm_HandSolder, symbol Device:R
Connections:
- net +5V: now also D2.2 (A), R1.1
- net GND: now also J1.7, D2.1 (K)
- net ~RDFE: now also U1.1 (PD3); no longer U1.32 (PD2)
- net ~RESET: now also U1.2 (PD4); no longer U1.23 (PC0)
- net at U1.8 (PB7/XTAL2), Y1.1: now also C3.1; no longer C2.1
- net at U1.7 (PB6/XTAL1), Y1.2: now also C2.1; no longer C3.1
- net at J3.4 (Pin_4): now also U1.26 (PC3); no longer U1.1 (PD3)
- net at U1.10 (PD6): now also SW1.1; no longer J3.7 (Pin_7)
- net at U1.11 (PD7): now also SW2.1; no longer J3.8 (Pin_8)
- net at J3.5 (Pin_5): now also U1.27 (PC4); no longer U1.2 (PD4)
- net at U1.24 (PC1): now also J3.2 (Pin_2); no longer SW1.1
- net at U1.25 (PC2): now also J3.3 (Pin_3); no longer SW2.1
- net at J1.1: now also U1.9 (PD5); no longer U1.27 (PC4)
- net at U1.28 (PC5): now also J3.6 (Pin_6); no longer J1.5
- net at J5.5 (Pin_5), U1.29 (PC6/~RESET): now also D1.1 (K)
- net at J3.1 (Pin_1): now also U1.23 (PC0); no longer U1.30 (PD0)
- net at U1.31 (PD1): now also J3.8 (Pin_8); no longer J3.2 (Pin_2)
- new net: J3.7 (Pin_7), U1.30 (PD0)
- new net: J1.5, U1.32 (PD2)
- new net: D1.2 (A), R1.2
Other:
- moved on the sheet: C1, C2, C3, J2, J3, J4, Y1

Commit message: Version 4 pre-production
Parts:
- added R2: 330Ω, Resistor_SMD:R_0805_2012Metric_Pad1.15x1.40mm_HandSolder, symbol Device:R
- J1: symbol Connector:Mini-DIN-6 -> ps2zx-rescue:Mini-DIN-6-Connector-ps2zx-rescue
Connections:
- net +5V: now also R2.1; no longer D2.2 (A)
- new net: D2.2 (A), R2.2
Changed lines of the file:
@@
 $EndComp
 $Comp
-L Connector:Mini-DIN-6 J1
+L ps2zx-rescue:Mini-DIN-6-Connector-ps2zx-rescue J1
 U 1 1 5EDFC7B4
 P 4850 2150
@@
 L power:+5V #PWR011
 U 1 1 5EF46876
-P 2250 4850
-F 0 "#PWR011" H 2250 4700 50  0001 C CNN
-F 1 "+5V" H 2265 5023 50  0000 C CNN
-F 2 "" H 2250 4850 50  0001 C CNN
-F 3 "" H 2250 4850 50  0001 C CNN
-	1    2250 4850
+P 2250 4550
+F 0 "#PWR011" H 2250 4400 50  0001 C CNN
+F 1 "+5V" H 2265 4723 50  0000 C CNN
+F 2 "" H 2250 4550 50  0001 C CNN
+F 3 "" H 2250 4550 50  0001 C CNN
+	1    2250 4550
 	1    0    0    -1
 $EndComp
@@
 	5250 1900 5150 1900
 Connection ~ 5250 2150
+$Comp
+L Device:R R2
+U 1 1 5EEFA480
+P 2250 4700
+F 0 "R2" H 2320 4746 50  0000 L CNN
+F 1 "330Ω" H 2320 4655 50  0000 L CNN
+F 2 "Resistor_SMD:R_0805_2012Metric_Pad1.15x1.40mm_HandSolder" V 2180 4700 50  0001 C CNN
+F 3 "~" H 2250 4700 50  0001 C CNN
+	1    2250 4700
+	1    0    0    -1
+$EndComp
 $EndSCHEMATC
